Commit message: Updated dofbot_arm_ctrl.urdf (noetic-devel)

File: dofbot_description/urdf/dofbot_arm_ctrl.urdf (robot description, URDF)
Before this commit: robot dofbot_arm, 13 links, 12 joints
Links:
- added link base_footprint
- link base_link: mass None -> 1.0754239466482
Joints:
- added joint base_footprint_joint: type fixed, parent base_footprint, child base_link
